File: PCBBoards/motorspeed.sch (EAGLE design)
At the start: 11 parts, among them IC1 LM358N, T1 2N2222

Commit message: Update PCB Board
Parts:
- removed X1: (no value), con-wago-500:W237-103
- removed X2: (no value), con-wago-500:W237-102
- added X3, X4: (no value), con-ptr500:AK500/3-H
Connections:
- removed net N$5: IC1A.-IN, IC1A.OUT
- new net SIG: IC1A.-IN, IC1A.OUT, X3-1.KL
- net +12V: now also X3-3.KL; no longer X2-1.KL
- net +5V: now also X4-1.KL; no longer X1-1.KL
- net 3.3V: now also X4-3.KL; no longer X1-3.KL
- net GND+12: now also X3-2.KL; no longer X2-2.KL
- net GND+3.3: now also X4-2.KL; no longer X1-2.KL
Changed lines of the file:
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@@
 <part name="R5" library="rcl" library_urn="urn:adsk.eagle:library:334" deviceset="R-EU_" device="0207/12" package3d_urn="urn:adsk.eagle:package:23489/1" value="10k"/>
 <part name="C1" library="rcl" library_urn="urn:adsk.eagle:library:334" deviceset="CPOL-EU" device="E2-5" package3d_urn="urn:adsk.eagle:package:23346/2" value="1u"/>
-<part name="X1" library="con-wago-500" library_urn="urn:adsk.eagle:library:195" deviceset="W237-103" device="" package3d_urn="urn:adsk.eagle:package:10691/1"/>
-<part name="X2" library="con-wago-500" library_urn="urn:adsk.eagle:library:195" deviceset="W237-102" device="" package3d_urn="urn:adsk.eagle:package:10688/1"/>
+<part name="X3" library="con-ptr500" library_urn="urn:adsk.eagle:library:181" deviceset="AK500/3-H" device="" package3d_urn="urn:adsk.eagle:package:9899/1"/>
+<part name="X4" library="con-ptr500" library_urn="urn:adsk.eagle:library:181" deviceset="AK500/3-H" device="" package3d_urn="urn:adsk.eagle:package:9899/1"/>
 </parts>
 <sheets>
@@
 <attribute name="VALUE" x="97.663" y="79.2226" size="1.778" layer="96"/>
 </instance>
-<instance part="X1" gate="-1" x="0" y="109.22" smashed="yes">
-<attribute name="NAME" x="0" y="110.109" size="1.778" layer="95" rot="R180"/>
-</instance>
-<instance part="X1" gate="-2" x="0" y="104.14" smashed="yes">
-<attribute name="NAME" x="0" y="105.029" size="1.778" layer="95" rot="R180"/>
-</instance>
-<instance part="X1" gate="-3" x="0" y="99.06" smashed="yes">
-<attribute name="VALUE" x="-2.54" y="95.377" size="1.778" layer="96"/>
-<attribute name="NAME" x="0" y="99.949" size="1.778" layer="95" rot="R180"/>
-</instance>
-<instance part="X2" gate="-1" x="-2.54" y="127" smashed="yes">
-<attribute name="NAME" x="-2.54" y="127.889" size="1.778" layer="95" rot="R180"/>
-</instance>
-<instance part="X2" gate="-2" x="-2.54" y="121.92" smashed="yes">
-<attribute name="VALUE" x="-5.08" y="118.237" size="1.778" layer="96"/>
-<attribute name="NAME" x="-2.54" y="122.809" size="1.778" layer="95" rot="R180"/>
-</instance>
 <instance part="IC1" gate="P" x="121.92" y="93.98" smashed="yes"/>
+<instance part="X3" gate="-1" x="40.64" y="144.78" smashed="yes">
+<attribute name="NAME" x="39.37" y="145.669" size="1.778" layer="95" rot="R180"/>
+</instance>
+<instance part="X3" gate="-2" x="40.64" y="139.7" smashed="yes">
+<attribute name="NAME" x="39.37" y="140.589" size="1.778" layer="95" rot="R180"/>
+</instance>
+<instance part="X3" gate="-3" x="40.64" y="134.62" smashed="yes">
+<attribute name="NAME" x="39.37" y="135.509" size="1.778" layer="95" rot="R180"/>
+<attribute name="VALUE" x="36.83" y="130.937" size="1.778" layer="96"/>
+</instance>
+<instance part="X4" gate="-1" x="7.62" y="129.54" smashed="yes">
+<attribute name="NAME" x="6.35" y="130.429" size="1.778" layer="95" rot="R180"/>
+</instance>
+<instance part="X4" gate="-2" x="7.62" y="124.46" smashed="yes">
+<attribute name="NAME" x="6.35" y="125.349" size="1.778" layer="95" rot="R180"/>
+</instance>
+<instance part="X4" gate="-3" x="7.62" y="119.38" smashed="yes">
+<attribute name="NAME" x="6.35" y="120.269" size="1.778" layer="95" rot="R180"/>
+<attribute name="VALUE" x="3.81" y="115.697" size="1.778" layer="96"/>
+</instance>
 </instances>
 <busses>
@@
 </segment>
 <segment>
-<pinref part="X2" gate="-1" pin="KL"/>
-<wire x1="2.54" y1="127" x2="7.62" y2="127" width="0.1524" layer="91"/>
-<label x="7.62" y="127" size="1.778" layer="95"/>
-</segment>
-<segment>
 <pinref part="IC1" gate="P" pin="V+"/>
 <wire x1="121.92" y1="101.6" x2="121.92" y2="106.68" width="0.1524" layer="91"/>
 <wire x1="121.92" y1="106.68" x2="127" y2="106.68" width="0.1524" layer="91"/>
 <label x="127" y="106.68" size="1.778" layer="95"/>
+</segment>
+<segment>
+<pinref part="X3" gate="-3" pin="KL"/>
+<wire x1="45.72" y1="134.62" x2="55.88" y2="134.62" width="0.1524" layer="91"/>
+<label x="58.42" y="134.62" size="1.778" layer="95"/>
 </segment>
 </net>
@@
 </segment>
 <segment>
-<pinref part="X2" gate="-2" pin="KL"/>
-<wire x1="2.54" y1="121.92" x2="7.62" y2="121.92" width="0.1524" layer="91"/>
-<label x="10.16" y="121.92" size="1.778" layer="95"/>
-</segment>
-<segment>
 <pinref part="IC1" gate="P" pin="V-"/>
 <wire x1="121.92" y1="86.36" x2="129.54" y2="86.36" width="0.1524" layer="91"/>
 <label x="132.08" y="86.36" size="1.778" layer="95"/>
 </segment>
-</net>
-<net name="N$5" class="0">
+<segment>
+<pinref part="X3" gate="-2" pin="KL"/>
+<wire x1="45.72" y1="139.7" x2="55.88" y2="139.7" width="0.1524" layer="91"/>
+<label x="58.42" y="139.7" size="1.778" layer="95"/>
+</segment>
+</net>
+<net name="SIG" class="0">
 <segment>
 <pinref part="IC1" gate="A" pin="OUT"/>
@@
 <wire x1="114.3" y1="81.28" x2="114.3" y2="91.44" width="0.1524" layer="91"/>
 <pinref part="IC1" gate="A" pin="-IN"/>
+<label x="137.16" y="96.52" size="1.778" layer="95"/>
+</segment>
+<segment>
+<pinref part="X3" gate="-1" pin="KL"/>
+<wire x1="45.72" y1="144.78" x2="55.88" y2="144.78" width="0.1524" layer="91"/>
+<label x="58.42" y="144.78" size="1.778" layer="95"/>
 </segment>
 </net>
@@
 </segment>
 <segment>
-<pinref part="X1" gate="-1" pin="KL"/>
-<wire x1="5.08" y1="109.22" x2="10.16" y2="109.22" width="0.1524" layer="91"/>
-<label x="12.7" y="109.22" size="1.778" layer="95"/>
+<pinref part="X4" gate="-1" pin="KL"/>
+<wire x1="12.7" y1="129.54" x2="20.32" y2="129.54" width="0.1524" layer="91"/>
+<label x="25.4" y="129.54" size="1.778" layer="95"/>
 </segment>
 </net>
 <net name="3.3V" class="0">
-<segment>
-<pinref part="X1" gate="-3" pin="KL"/>
-<wire x1="5.08" y1="99.06" x2="10.16" y2="99.06" width="0.1524" layer="91"/>
-<label x="12.7" y="99.06" size="1.778" layer="95"/>
-</segment>
 <segment>
 <pinref part="R5" gate="G$1" pin="1"/>
 <wire x1="12.7" y1="83.82" x2="5.08" y2="83.82" width="0.1524" layer="91"/>
 <label x="2.54" y="86.36" size="1.778" layer="95"/>
+</segment>
+<segment>
+<pinref part="X4" gate="-3" pin="KL"/>
+<wire x1="12.7" y1="119.38" x2="20.32" y2="119.38" width="0.1524" layer="91"/>
+<label x="25.4" y="119.38" size="1.778" layer="95"/>
 </segment>
 </net>
@@
 </segment>
 <segment>
-<pinref part="X1" gate="-2" pin="KL"/>
-<wire x1="5.08" y1="104.14" x2="10.16" y2="104.14" width="0.1524" layer="91"/>
-<label x="12.7" y="104.14" size="1.778" layer="95"/>
-</segment>
-</net>
+<pinref part="X4" gate="-2" pin="KL"/>
+<wire x1="12.7" y1="124.46" x2="20.32" y2="124.46" width="0.1524" layer="91"/>
+<label x="25.4" y="124.46" size="1.778" layer="95"/>
+</segment>
+</net>
