File: PCBBoards/motorspeed.brd (EAGLE design)
At the start: 27.4 x 40.8 mm, 11 parts, among them IC1 LM358N, T1 2N2222

Commit message: Update PCB Board
Parts:
- removed X1: (no value), con-wago-500:W237-103
- removed X2: (no value), con-wago-500:W237-102
- added X3, X4: (no value), con-ptr500:AK500/3-H
Connections:
- removed net N$5: IC1.1, IC1.2
- new net SIG: IC1.1, IC1.2, X3.1
- net +12V: now also X3.3; no longer X2.1
- net +5V: now also X4.1; no longer X1.1
- net 3.3V: now also X4.3; no longer X1.3
- net GND+12: now also X3.2; no longer X2.2
- net GND+3.3: now also X4.2; no longer X1.2
Routing:
- net SIG: track 0.00 -> 44.1 mm
- net GND+12: track 42.7 -> 47.9 mm
- net N$5: track 2.43 -> 0.00 mm
- net GND+3.3: track 10.2 -> 8.19 mm
- net 3.3V: track 7.45 -> 5.45 mm
- net +5V: track 7.29 -> 5.39 mm
- net +12V: track 33.0 -> 34.6 mm
- net N$7: track 10.3 -> 9.49 mm
Changed lines of the file:
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@@
 <attribute name="VALUE" x="-1.397" y="21.717" size="1.27" layer="27" ratio="10" rot="R90"/>
 </element>
-<element name="X1" library="con-wago-500" library_urn="urn:adsk.eagle:library:195" package="W237-103" package3d_urn="urn:adsk.eagle:package:10691/1" value="" x="8.128" y="6.096" smashed="yes">
-<attribute name="MF" value="" x="38.608" y="-2.794" size="1.778" layer="27" display="off"/>
-<attribute name="MPN" value="237-103" x="38.608" y="-2.794" size="1.778" layer="27" display="off"/>
-<attribute name="NAME" x="16.4122" y="2.4438" size="1.27" layer="25" ratio="10"/>
-<attribute name="OC_FARNELL" value="unknown" x="38.608" y="-2.794" size="1.778" layer="27" display="off"/>
-<attribute name="OC_NEWARK" value="18M7116" x="38.608" y="-2.794" size="1.778" layer="27" display="off"/>
-<attribute name="VALUE" x="2.8232" y="1.1484" size="1.27" layer="27" ratio="10"/>
+<element name="X3" library="con-ptr500" library_urn="urn:adsk.eagle:library:181" package="AK500/3-H" package3d_urn="urn:adsk.eagle:package:9899/1" value="" x="20.32" y="32.766" smashed="yes" rot="R90">
+<attribute name="MF" value="" x="20.32" y="32.766" size="1.778" layer="27" rot="R90" display="off"/>
+<attribute name="MPN" value="" x="20.32" y="32.766" size="1.778" layer="27" rot="R90" display="off"/>
+<attribute name="NAME" x="16.764" y="25.1714" size="1.778" layer="25" ratio="10" rot="R90"/>
+<attribute name="OC_FARNELL" value="unknown" x="20.32" y="32.766" size="1.778" layer="27" rot="R90" display="off"/>
+<attribute name="OC_NEWARK" value="unknown" x="20.32" y="32.766" size="1.778" layer="27" rot="R90" display="off"/>
+<attribute name="VALUE" x="29.845" y="25.1714" size="1.778" layer="27" ratio="10" rot="R90"/>
 </element>
-<element name="X2" library="con-wago-500" library_urn="urn:adsk.eagle:library:195" package="W237-102" package3d_urn="urn:adsk.eagle:package:10688/1" value="" x="22.86" y="32.766" smashed="yes" rot="R270">
-<attribute name="MF" value="" x="3.81" y="14.986" size="1.778" layer="27" rot="R270" display="off"/>
-<attribute name="MPN" value="237-102" x="3.81" y="14.986" size="1.778" layer="27" rot="R270" display="off"/>
-<attribute name="NAME" x="0.4718" y="56.7182" size="1.27" layer="25" ratio="10"/>
-<attribute name="OC_FARNELL" value="unknown" x="3.81" y="14.986" size="1.778" layer="27" rot="R270" display="off"/>
-<attribute name="OC_NEWARK" value="70K9898" x="3.81" y="14.986" size="1.778" layer="27" rot="R270" display="off"/>
-<attribute name="VALUE" x="15.24" y="37.806" size="1.27" layer="27" ratio="10" rot="R270"/>
+<element name="X4" library="con-ptr500" library_urn="urn:adsk.eagle:library:181" package="AK500/3-H" package3d_urn="urn:adsk.eagle:package:9899/1" value="" x="8.128" y="6.858" smashed="yes">
+<attribute name="MF" value="" x="8.128" y="6.858" size="1.778" layer="27" display="off"/>
+<attribute name="MPN" value="" x="8.128" y="6.858" size="1.778" layer="27" display="off"/>
+<attribute name="NAME" x="0.5334" y="10.414" size="1.778" layer="25" ratio="10"/>
+<attribute name="OC_FARNELL" value="unknown" x="8.128" y="6.858" size="1.778" layer="27" display="off"/>
+<attribute name="OC_NEWARK" value="unknown" x="8.128" y="6.858" size="1.778" layer="27" display="off"/>
+<attribute name="VALUE" x="0.5334" y="-2.667" size="1.778" layer="27" ratio="10"/>
 </element>
 </elements>
@@
 <signal name="+12V">
 <contactref element="R3" pad="2"/>
-<contactref element="X2" pad="1"/>
-<wire x1="16.58221875" y1="37.06258125" x2="14.986" y2="38.6588" width="0.1524" layer="1"/>
-<wire x1="14.986" y1="38.862" x2="14.986" y2="38.6588" width="0.1524" layer="1"/>
-<wire x1="16.58221875" y1="37.06258125" x2="21.59" y2="35.266" width="0.1524" layer="1"/>
 <contactref element="IC1" pad="8"/>
-<wire x1="25.654" y1="11.176" x2="25.654" y2="29.92385" width="0.1524" layer="1"/>
-<wire x1="25.654" y1="29.92385" x2="21.0692875" y2="34.5085625" width="0.1524" layer="1"/>
-<wire x1="21.0692875" y1="34.5085625" x2="21.59" y2="35.266" width="0" layer="19" extent="1-1"/>
+<contactref element="X3" pad="3"/>
+<wire x1="14.986" y1="38.862" x2="19.2278" y2="38.862" width="0.1524" layer="1"/>
+<wire x1="19.2278" y1="38.862" x2="20.32" y2="37.7698" width="0.1524" layer="1"/>
+<wire x1="20.32" y1="37.7698" x2="23.876" y2="34.2138" width="0.1524" layer="1"/>
+<wire x1="25.654" y1="13.716" x2="25.654" y2="11.176" width="0.1524" layer="1"/>
+<wire x1="23.876" y1="34.2138" x2="23.876" y2="15.494" width="0.1524" layer="1"/>
+<wire x1="23.876" y1="15.494" x2="25.654" y2="13.716" width="0.1524" layer="1"/>
 </signal>
 <signal name="N$2">
@@
 <contactref element="C1" pad="-"/>
 <contactref element="R2" pad="2"/>
-<contactref element="X2" pad="2"/>
-<wire x1="19.6596" y1="29.506" x2="19.6596" y2="26.416" width="0.1524" layer="1"/>
-<wire x1="19.6596" y1="29.506" x2="21.59" y2="30.266" width="0.1524" layer="1"/>
-<wire x1="11.8872" y1="23.9268" x2="11.3182375" y2="23.64231875" width="0.1524" layer="1"/>
 <wire x1="11.176" y1="23.622" x2="11.3182375" y2="23.64231875" width="0.1524" layer="1"/>
 <wire x1="11.176" y1="23.622" x2="13.97" y2="26.416" width="0.1524" layer="1"/>
-<wire x1="13.97" y1="26.416" x2="19.6596" y2="26.416" width="0.1524" layer="1"/>
+<wire x1="13.97" y1="26.416" x2="16.002" y2="26.416" width="0.1524" layer="1"/>
 <contactref element="IC1" pad="4"/>
+<wire x1="16.002" y1="26.416" x2="19.6596" y2="26.416" width="0.1524" layer="1"/>
 <wire x1="18.034" y1="3.556" x2="22.86" y2="8.382" width="0.1524" layer="1"/>
 <wire x1="22.86" y1="8.382" x2="22.86" y2="19.304" width="0.1524" layer="1"/>
@@
 <wire x1="22.86" y1="19.304" x2="21.59" y2="20.574" width="0.1524" layer="1"/>
 <wire x1="21.59" y1="20.574" x2="20.066" y2="20.574" width="0.1524" layer="1"/>
+<contactref element="X3" pad="2"/>
+<wire x1="16.002" y1="26.416" x2="16.002" y2="33.02" width="0.1524" layer="1"/>
+<wire x1="16.002" y1="33.02" x2="20.066" y2="33.02" width="0.1524" layer="1"/>
+<wire x1="20.066" y1="33.02" x2="20.32" y2="32.766" width="0.1524" layer="1"/>
 </signal>
-<signal name="N$5">
+<signal name="SIG">
 <contactref element="IC1" pad="1"/>
 <contactref element="IC1" pad="2"/>
@@
 <wire x1="18.1356" y1="8.636" x2="18.034" y2="8.636" width="0.1524" layer="1"/>
 <wire x1="18.1356" y1="11.0744" x2="18.034" y2="11.176" width="0.1524" layer="1"/>
+<contactref element="X3" pad="1"/>
+<wire x1="18.034" y1="11.176" x2="16.51" y2="9.652" width="0.1524" layer="1"/>
+<wire x1="16.51" y1="9.652" x2="16.51" y2="3.048" width="0.1524" layer="1"/>
+<wire x1="16.51" y1="3.048" x2="17.78" y2="1.778" width="0.1524" layer="1"/>
+<wire x1="17.78" y1="1.778" x2="24.257" y2="8.255" width="0.1524" layer="1"/>
+<wire x1="24.257" y1="14.68194375" x2="24.257" y2="8.255" width="0.1524" layer="1"/>
+<wire x1="21.7678" y1="27.7622" x2="23.368" y2="26.162" width="0.1524" layer="1"/>
+<wire x1="21.7678" y1="27.7622" x2="20.32" y2="27.7622" width="0.1524" layer="1"/>
+<wire x1="23.368" y1="15.57094375" x2="24.257" y2="14.68194375" width="0.1524" layer="1"/>
+<wire x1="23.368" y1="26.162" x2="23.368" y2="15.57094375" width="0.1524" layer="1"/>
+<wire x1="18.1356" y1="11.0744" x2="18.1356" y2="10.8204" width="0" layer="19" extent="1-1"/>
 </signal>
 <signal name="N$6">
@@
 <contactref element="T1" pad="2"/>
 <contactref element="R5" pad="2"/>
-<wire x1="8.6868" y1="17.5768" x2="8.6868" y2="16.6116" width="0.1524" layer="1"/>
-<wire x1="15.24" y1="24.13" x2="8.6868" y2="17.5768" width="0.1524" layer="1"/>
-<wire x1="8.9408" y1="17.3736" x2="8.89" y2="17.272" width="0.1524" layer="1"/>
+<wire x1="15.24" y1="24.13" x2="8.89" y2="17.78" width="0.1524" layer="1"/>
+<wire x1="8.89" y1="17.78" x2="8.89" y2="17.272" width="0.1524" layer="1"/>
 </signal>
 <signal name="N$8">
@@
 <signal name="+5V">
 <contactref element="R4" pad="1"/>
-<contactref element="X1" pad="1"/>
-<wire x1="2.1336" y1="6.096" x2="2.1336" y2="11.6332" width="0.1524" layer="1"/>
-<wire x1="2.5595375" y1="5.6700625" x2="2.1336" y2="6.096" width="0.1524" layer="1"/>
 <wire x1="2.1336" y1="11.6332" x2="2.032" y2="11.684" width="0.1524" layer="1"/>
-<wire x1="2.5595375" y1="5.6700625" x2="3.128" y2="4.806" width="0.1524" layer="1"/>
+<contactref element="X4" pad="1"/>
+<wire x1="2.032" y1="11.684" x2="2.032" y2="8.128" width="0.1524" layer="1"/>
+<wire x1="2.032" y1="8.128" x2="3.1242" y2="7.0358" width="0.1524" layer="1"/>
+<wire x1="3.1242" y1="7.0358" x2="3.1242" y2="6.858" width="0.1524" layer="1"/>
 </signal>
 <signal name="3.3V">
-<contactref element="X1" pad="3"/>
 <contactref element="R5" pad="1"/>
-<wire x1="15.24" y1="7.278109375" x2="15.24" y2="11.43" width="0.1524" layer="1"/>
-<wire x1="15.24" y1="7.278109375" x2="13.128" y2="5.0063125" width="0.1524" layer="1"/>
-<wire x1="13.128" y1="4.806" x2="13.128" y2="5.0063125" width="0.1524" layer="1"/>
+<contactref element="X4" pad="3"/>
+<wire x1="15.24" y1="11.43" x2="15.24" y2="8.9662" width="0.1524" layer="1"/>
+<wire x1="15.24" y1="8.9662" x2="13.1318" y2="6.858" width="0.1524" layer="1"/>
 </signal>
 <signal name="GND+3.3">
 <contactref element="T1" pad="1"/>
-<contactref element="X1" pad="2"/>
-<wire x1="8.5344" y1="5.4864" x2="8.5344" y2="14.3764" width="0.1524" layer="1"/>
-<wire x1="8.5344" y1="14.3764" x2="8.89" y2="14.732" width="0.1524" layer="1"/>
-<wire x1="8.5344" y1="5.4864" x2="8.128" y2="5" width="0.1524" layer="1"/>
-<wire x1="8.128" y1="4.806" x2="8.128" y2="5" width="0.1524" layer="1"/>
+<contactref element="X4" pad="2"/>
+<wire x1="8.128" y1="6.858" x2="8.128" y2="10.414" width="0.1524" layer="1"/>
+<wire x1="8.128" y1="10.414" x2="8.89" y2="11.176" width="0.1524" layer="1"/>
+<wire x1="8.89" y1="11.176" x2="8.89" y2="14.732" width="0.1524" layer="1"/>
 </signal>
 </signals>

Commit message: Update motorspeed.brd
Parts:
- moved T1 0.80 mm to (6.86, 16.3)
Routing:
- net GND+12: track 47.9 -> 0.14 mm
- net N$6: track 11.4 -> 10.6 mm
- added copper zone on layer 1, net GND+12
Changed lines of the file:
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@@
 <attribute name="VALUE" x="15.6718" y="16.51" size="1.27" layer="27" ratio="10" rot="R90"/>
 </element>
-<element name="T1" library="transistor" library_urn="urn:adsk.eagle:library:402" package="TO18" package3d_urn="urn:adsk.eagle:package:28526/2" value="2N2222" x="7.62" y="16.002" smashed="yes" rot="R90">
-<attribute name="NAME" x="-1.778" y="14.605" size="1.27" layer="25" ratio="10" rot="R90"/>
-<attribute name="VALUE" x="-1.397" y="21.717" size="1.27" layer="27" ratio="10" rot="R90"/>
+<element name="T1" library="transistor" library_urn="urn:adsk.eagle:library:402" package="TO18" package3d_urn="urn:adsk.eagle:package:28526/2" value="2N2222" x="6.858" y="16.256" smashed="yes" rot="R90">
+<attribute name="NAME" x="-2.54" y="14.859" size="1.27" layer="25" ratio="10" rot="R90"/>
+<attribute name="VALUE" x="-2.159" y="21.971" size="1.27" layer="27" ratio="10" rot="R90"/>
 </element>
 <element name="X3" library="con-ptr500" library_urn="urn:adsk.eagle:library:181" package="AK500/3-H" package3d_urn="urn:adsk.eagle:package:9899/1" value="" x="20.32" y="32.766" smashed="yes" rot="R90">
@@
 <contactref element="R2" pad="2"/>
 <wire x1="11.176" y1="23.622" x2="11.3182375" y2="23.64231875" width="0.1524" layer="1"/>
-<wire x1="11.176" y1="23.622" x2="13.97" y2="26.416" width="0.1524" layer="1"/>
-<wire x1="13.97" y1="26.416" x2="16.002" y2="26.416" width="0.1524" layer="1"/>
 <contactref element="IC1" pad="4"/>
-<wire x1="16.002" y1="26.416" x2="19.6596" y2="26.416" width="0.1524" layer="1"/>
-<wire x1="18.034" y1="3.556" x2="22.86" y2="8.382" width="0.1524" layer="1"/>
-<wire x1="22.86" y1="8.382" x2="22.86" y2="19.304" width="0.1524" layer="1"/>
-<wire x1="19.6596" y1="26.416" x2="19.6596" y2="20.9804" width="0.1524" layer="1"/>
-<wire x1="19.6596" y1="20.9804" x2="20.066" y2="20.574" width="0.1524" layer="1"/>
-<wire x1="22.86" y1="19.304" x2="21.59" y2="20.574" width="0.1524" layer="1"/>
-<wire x1="21.59" y1="20.574" x2="20.066" y2="20.574" width="0.1524" layer="1"/>
 <contactref element="X3" pad="2"/>
-<wire x1="16.002" y1="26.416" x2="16.002" y2="33.02" width="0.1524" layer="1"/>
-<wire x1="16.002" y1="33.02" x2="20.066" y2="33.02" width="0.1524" layer="1"/>
-<wire x1="20.066" y1="33.02" x2="20.32" y2="32.766" width="0.1524" layer="1"/>
+<polygon width="0.1524" layer="1">
+<vertex x="0" y="41.148"/>
+<vertex x="0" y="-0.254"/>
+<vertex x="27.686" y="-0.254"/>
+<vertex x="27.686" y="41.148"/>
+</polygon>
+<wire x1="20.066" y1="20.574" x2="20.32" y2="32.766" width="0" layer="19" extent="1-1"/>
+<wire x1="11.3182375" y1="23.64231875" x2="20.066" y2="20.574" width="0" layer="19" extent="1-1"/>
+<wire x1="18.034" y1="3.556" x2="20.066" y2="20.574" width="0" layer="19" extent="1-1"/>
 </signal>
 <signal name="SIG">
@@
 <contactref element="OK1" pad="2"/>
 <wire x1="4.572" y1="18.1356" x2="4.572" y2="27.432" width="0.1524" layer="1"/>
-<wire x1="5.4356" y1="17.272" x2="4.572" y2="18.1356" width="0.1524" layer="1"/>
-<wire x1="5.4356" y1="17.272" x2="6.35" y2="17.272" width="0.1524" layer="1"/>
+<wire x1="5.1816" y1="17.526" x2="4.572" y2="18.1356" width="0.1524" layer="1"/>
+<wire x1="5.1816" y1="17.526" x2="5.588" y2="17.526" width="0.1524" layer="1"/>
 </signal>
 <signal name="N$7">
 <contactref element="T1" pad="2"/>
 <contactref element="R5" pad="2"/>
-<wire x1="15.24" y1="24.13" x2="8.89" y2="17.78" width="0.1524" layer="1"/>
-<wire x1="8.89" y1="17.78" x2="8.89" y2="17.272" width="0.1524" layer="1"/>
+<wire x1="15.24" y1="24.13" x2="8.636" y2="17.526" width="0.1524" layer="1"/>
+<wire x1="8.636" y1="17.526" x2="8.128" y2="17.526" width="0.1524" layer="1"/>
 </signal>
 <signal name="N$8">
@@
 <wire x1="2.1336" y1="24.4348" x2="2.032" y2="24.384" width="0.1524" layer="1"/>
 <wire x1="2.1336" y1="27.3304" x2="2.032" y2="27.432" width="0.1524" layer="1"/>
+<wire x1="2.1336" y1="24.4348" x2="2.1336" y2="24.6888" width="0" layer="19" extent="1-1"/>
 </signal>
 <signal name="+5V">
@@
 <contactref element="T1" pad="1"/>
 <contactref element="X4" pad="2"/>
-<wire x1="8.128" y1="6.858" x2="8.128" y2="10.414" width="0.1524" layer="1"/>
-<wire x1="8.128" y1="10.414" x2="8.89" y2="11.176" width="0.1524" layer="1"/>
-<wire x1="8.89" y1="11.176" x2="8.89" y2="14.732" width="0.1524" layer="1"/>
+<wire x1="8.128" y1="6.858" x2="8.128" y2="14.986" width="0.1524" layer="1"/>
 </signal>
 </signals>

Commit message: final version
Routing:
- net SIG: track 44.1 -> 22.8 mm
- net N$3: track 33.1 -> 34.6 mm
- net N$2: track 7.94 -> 7.34 mm
