File: PCBBoards/demux.sch (EAGLE design)
At the start: 79 parts, among them IC1 4013N, IC2 4013N, IC3 4013N, IC4 4013N, IC5 4013N, IC6 4013N, IC7 4069N, IC8 4069N, Q1 2N3904, Q10 2N3904, Q11 2N3904, Q12 2N3904, Q2 2N3904, Q3 2N3904, Q4 2N3904, Q5 2N3904, Q6 2N3904, Q7 2N3904, Q8 2N3904, Q9 2N3904

Commit message: fr/sr update
Connections:
- removed net +3V31: R20.2
- net +3V3: now also R20.2
Changed lines of the file:
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@@
 <attribute name="VALUE" x="320.04" y="-48.26" size="1.778" layer="96"/>
 </instance>
-<instance part="+3V1" gate="G$1" x="388.62" y="165.1" smashed="yes" rot="R270">
-<attribute name="VALUE" x="383.54" y="167.64" size="1.778" layer="96"/>
+<instance part="+3V1" gate="G$1" x="386.08" y="165.1" smashed="yes" rot="R270">
+<attribute name="VALUE" x="381" y="167.64" size="1.778" layer="96"/>
 </instance>
 <instance part="+3V2" gate="G$1" x="386.08" y="124.46" smashed="yes" rot="R270">
@@
 <label x="396.24" y="165.1" size="1.778" layer="95"/>
 </segment>
+<segment>
+<pinref part="R20" gate="G$1" pin="2"/>
+<pinref part="+3V1" gate="G$1" pin="+3V3"/>
+<wire x1="383.54" y1="165.1" x2="375.92" y2="165.1" width="0.1524" layer="91"/>
+</segment>
 </net>
 <net name="N$65" class="0">
@@
 </segment>
 </net>
-<net name="+3V31" class="0">
-<segment>
-<pinref part="R20" gate="G$1" pin="2"/>
-<pinref part="+3V1" gate="G$1" pin="+3V3"/>
-<wire x1="386.08" y1="165.1" x2="375.92" y2="165.1" width="0.1524" layer="91"/>
-</segment>
-</net>

Commit message: Add needed elements
Parts:
- added C1, C2, C3, C4, C5, C6, C7, C8, C9: 100n, rcl:C-EU050-035X075
- added R37, R39, R41, R43, R45, R47: 10k, rcl:R-EU_0207/10
- added R38, R40, R42, R44, R46, R48: 260k, rcl:R-EU_0207/10
- added T1, T2, T3, T4, T5, T6: 2N3904, transistor-neu-to92:2N3904
Connections:
- new net IN_0: R37.1, T1.C, V11.A
- new net IN_1: R39.1, T2.C, V11.B
- new net IN_2: R43.1, T4.C, V11.C
- new net IN_3: R41.1, T3.C, V11.D
- new net IN_4: R45.1, T5.C, V11.!G1, V11.!G2
- new net IN_5: IC1A.R, IC1B.R, IC2A.R, IC2B.R, IC3A.R, IC3B.R, IC4A.R, IC4B.R, IC5A.R, IC5B.R, IC6A.R, IC6B.R, R47.1, T6.C
- new net N$63: R40.1, T2.B
- new net N$70: R38.1, T1.B
- new net N$73: R42.1, T3.B
- new net N$75: R44.1, T4.B
- new net N$77: R46.1, T5.B
- new net N$79: R48.1, T6.B
- net +5V: now also C1.1, C2.1, C3.1, C4.1, C5.1, C6.1, C7.2, C8.1, C9.1, R37.2, R39.2, R41.2, R43.2, R45.2, R47.2
- net GND: now also C1.2, C2.2, C3.2, C4.2, C5.2, C6.2, C7.1, C8.2, C9.2, IC1A.S, IC1B.S, IC2A.S, IC2B.S, IC3A.S, IC3B.S, IC4A.S, IC4B.S, IC5A.S, IC5B.S, IC6A.S, IC6B.S, T1.E, T2.E, T3.E, T4.E, T5.E, T6.E
- net GPIO1: now also R38.2; no longer V11.A
- net GPIO2: now also R40.2; no longer V11.B
- net GPIO3: now also R44.2; no longer V11.C
- net GPIO4: now also R42.2; no longer V11.D
- net GPIO5: now also R46.2; no longer V11.!G1, V11.!G2
- net GPIO6: now also R48.2; no longer IC1A.R, IC1A.S, IC1B.R, IC1B.S, IC2A.R, IC2A.S, IC2B.R, IC2B.S, IC3A.R, IC3A.S, IC3B.R, IC3B.S, IC4A.R, IC4A.S, IC4B.R, IC4B.S, IC5A.R, IC5A.S, IC5B.R, IC5B.S, IC6A.R, IC6A.S, IC6B.R, IC6B.S
Other:
- moved on the sheet: IC1P, IC2P, IC3P, IC4P, IC5P, IC6P, IC7P, IC8P, R34, R36, V1/+UB, V1/-UB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
