File: PCBBoards/demux.brd (EAGLE design)
At the start: 160 x 100 mm, 79 parts, among them IC1 4013N, IC2 4013N, IC3 4013N, IC4 4013N, IC5 4013N, IC6 4013N, IC7 4069N, IC8 4069N, Q1 2N3904, Q10 2N3904, Q11 2N3904, Q12 2N3904, Q2 2N3904, Q3 2N3904, Q4 2N3904, Q5 2N3904, Q6 2N3904, Q7 2N3904, Q8 2N3904, Q9 2N3904

Commit message: fr/sr update
Parts:
- moved R36 336.3 mm to (156.2, -41.9), turned to 90 degrees
- moved R35 329.5 mm to (151.1, -41.9), turned to 90 degrees
- moved R34 322.7 mm to (146.1, -41.9), turned to 90 degrees
- moved X16 322.6 mm to (144.8, -64.8)
- moved R33 316.0 mm to (141.0, -41.9), turned to 90 degrees
- moved R32 309.2 mm to (135.9, -41.9), turned to 90 degrees
- moved R31 302.5 mm to (130.8, -41.9), turned to 90 degrees
- moved OK6 299.6 mm to (137.2, 8.89), turned to 180 degrees
- moved R30 295.8 mm to (125.7, -41.9), turned to 90 degrees
- moved R29 289.2 mm to (120.7, -41.9), turned to 90 degrees
- moved X15 287.4 mm to (111.8, -64.8)
- moved R28 282.5 mm to (115.6, -41.9), turned to 90 degrees
- moved OK5 280.3 mm to (127.0, 8.89), turned to 180 degrees
- moved R27 275.9 mm to (110.5, -41.9), turned to 90 degrees
- moved X14 274.9 mm to (128.3, -64.8)
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Connections:
- removed net +3V31: R20.2
- net +3V3: now also R20.2
Other:
- board size 160 x 100 mm -> 168.9 x 169.8 mm

Commit message: Add needed elements
Parts:
- added C1, C2, C3, C4, C5, C6, C7, C8, C9: 100n, rcl:C050-035X075
- added R37, R39, R41, R43, R45, R47: 10k, rcl:0207/10
- added R38, R40, R42, R44, R46, R48: 260k, rcl:0207/10
- added T1, T2, T3, T4, T5, T6: 2N3904, transistor-neu-to92:TO92
Connections:
- new net IN_0: R37.1, T1.1, V1.23
- new net IN_1: R39.1, T2.1, V1.22
- new net IN_2: R43.1, T4.1, V1.21
- new net IN_3: R41.1, T3.1, V1.20
- new net IN_4: R45.1, T5.1, V1.18, V1.19
- new net IN_5: IC1.10, IC1.4, IC2.10, IC2.4, IC3.10, IC3.4, IC4.10, IC4.4, IC5.10, IC5.4, IC6.10, IC6.4, R47.1, T6.1
- new net N$63: R40.1, T2.2
- new net N$70: R38.1, T1.2
- new net N$73: R42.1, T3.2
- new net N$75: R44.1, T4.2
- new net N$77: R46.1, T5.2
- new net N$79: R48.1, T6.2
- net +5V: now also C1.1, C2.1, C3.1, C4.1, C5.1, C6.1, C7.2, C8.1, C9.1, R37.2, R39.2, R41.2, R43.2, R45.2, R47.2
- net GND: now also C1.2, C2.2, C3.2, C4.2, C5.2, C6.2, C7.1, C8.2, C9.2, IC1.6, IC1.8, IC2.6, IC2.8, IC3.6, IC3.8, IC4.6, IC4.8, IC5.6, IC5.8, IC6.6, IC6.8, T1.3, T2.3, T3.3, T4.3, T5.3, T6.3
- net GPIO1: now also R38.2; no longer V1.23
- net GPIO2: now also R40.2; no longer V1.22
- net GPIO3: now also R44.2; no longer V1.21
- net GPIO4: now also R42.2; no longer V1.20
- net GPIO5: now also R46.2; no longer V1.18, V1.19
- net GPIO6: now also R48.2; no longer IC1.10, IC1.4, IC1.6, IC1.8, IC2.10, IC2.4, IC2.6, IC2.8, IC3.10, IC3.4, IC3.6, IC3.8, IC4.10, IC4.4, IC4.6, IC4.8, IC5.10, IC5.4, IC5.6, IC5.8, IC6.10, IC6.4, IC6.6, IC6.8

Commit message: fr/sr another one
Parts:
- removed C2, C3, C4, C5, C6, C7, C8, C9: 100n, rcl:C050-035X075
- C1: value 100n -> 1u
- moved T6 203.0 mm to (26.7, 3.81), turned to 90 degrees
- moved R47 200.5 mm to (39.4, 5.08)
- moved T5 195.5 mm to (30.5, 8.89), turned to 90 degrees
- moved R48 191.6 mm to (16.5, 3.81), turned to 180 degrees
- moved R45 191.3 mm to (39.4, 10.2)
- moved R46 181.6 mm to (16.5, 8.89), turned to 180 degrees
- moved T3 170.8 mm to (26.7, 14.0), turned to 90 degrees
- moved R41 169.8 mm to (39.4, 15.2), flipped to the bottom
- moved T4 163.0 mm to (26.7, -12.7), turned to 90 degrees
- moved R43 162.5 mm to (39.4, -11.4)
- moved R42 158.3 mm to (16.5, 14.0), flipped to the bottom
- moved R9 154.3 mm to (5.08, 76.2), turned to 90 degrees
- moved R44 150.2 mm to (16.5, -12.7), turned to 180 degrees
- moved T2 145.9 mm to (30.5, -7.62), turned to 90 degrees
- moved R39 144.3 mm to (39.4, -6.35)
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Connections:
- new net N$80: IC6.11, IC8.8
- new net N$81: IC8.9
- net +5V: no longer C2.1, C3.1, C4.1, C5.1, C6.1, C7.2, C8.1, C9.1
- net GND: no longer C2.2, C3.2, C4.2, C5.2, C6.2, C7.1, C8.2, C9.2
- net N$11: now also IC5.11; no longer IC6.11
- net N$2: now also IC7.12; no longer IC7.8
- net N$27: now also IC7.13; no longer IC7.9
- net N$29: now also IC7.9; no longer IC7.13
- net N$33: no longer IC8.9
- net N$35: no longer IC8.13
- net N$5: now also IC7.8; no longer IC7.12
- net N$9: now also IC8.13; no longer IC5.11, IC8.8
Routing:
- net +5V: track 0.00 -> 330.4 mm, vias 0 -> 1
- net IN_5: track 0.00 -> 184.5 mm
- net FREQ2: track 0.00 -> 146.5 mm
- net GND_AKU: track 0.00 -> 117.4 mm
- net +3V3: track 0.00 -> 91.1 mm
- net N$32: track 0.00 -> 86.0 mm
- net IN_2: track 0.00 -> 83.3 mm, vias 0 -> 1
- net IN_1: track 0.00 -> 72.9 mm
- net N$34: track 0.00 -> 72.4 mm
- net IN_0: track 0.00 -> 70.7 mm, vias 0 -> 1
- net N$64: track 0.00 -> 57.2 mm
- net N$66: track 0.00 -> 55.4 mm
- net IN_3: track 0.00 -> 52.3 mm, vias 0 -> 1
- net N$31: track 0.00 -> 50.0 mm
- net IN_4: track 0.00 -> 47.8 mm
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- added copper zone on layer 1, net GND
Other:
- board size 168.9 x 169.8 mm -> 114.3 x 169.8 mm

Commit message: first version of complited FR/SR PCB board
Parts:
- moved C1 23.2 mm to (97.8, 11.4)
- moved X9 20.3 mm to (109.2, 11.4)
- moved IC5 17.8 mm to (26.7, 57.1)
- moved IC6 17.8 mm to (8.89, 57.1)
- moved Q10 17.8 mm to (30.5, 87.6)
- moved Q11 17.8 mm to (6.35, 87.6)
- moved Q12 17.8 mm to (12.7, 87.6)
- moved Q9 17.8 mm to (24.1, 87.6)
- moved R10 17.8 mm to (30.5, 76.2)
- moved R11 17.8 mm to (5.08, 76.2)
- moved R12 17.8 mm to (12.7, 76.2)
- moved R9 17.8 mm to (22.9, 76.2)
- moved X7 17.8 mm to (26.7, 95.2)
- moved X8 17.8 mm to (8.89, 95.2)
- moved R15 16.7 mm to (97.8, -6.35)
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Connections:
- removed net N$24: IC7.1, V1.1
- removed net N$3 (its old number): IC2.3, IC7.6
- removed net N$80: IC6.11, IC8.8
- removed net N$81: IC8.9
- new net N$4: IC1.3, IC7.10
- new net N$82: IC8.11, V1.9
- net N$1: now also IC2.3, IC7.12; no longer IC3.3, IC7.10
- net N$10: now also IC8.3, V1.10; no longer IC6.3, IC8.10
- net N$11: now also IC6.3, IC8.8; no longer IC5.11, IC8.12
- net N$13: now also IC3.11, IC7.6; no longer IC1.3, IC7.2
- net N$2: now also IC7.2; no longer IC7.12
- net N$26: now also IC7.13; no longer IC7.5
- net N$27: now also IC7.1; no longer IC7.13
- net N$28: now also IC7.9; no longer IC7.11
- net N$29: now also IC7.5; no longer IC7.9
- net N$30: now also IC8.13; no longer IC8.1
- net N$31: now also IC8.1; no longer IC8.3
- net N$32: now also IC5.11, IC8.4; no longer IC8.5, V1.9
- net N$33: now also IC5.3, IC8.10; no longer V1.10
- net N$34: now also IC8.9; no longer IC8.11
- net N$35: now also IC8.5
- net N$5: now also IC7.11, V1.1; no longer IC3.11, IC7.8
- net N$6: now also IC8.12; no longer IC8.2
- net N$7: now also IC8.2; no longer IC8.4
- net N$8: now also IC3.3, IC7.8; no longer IC5.3, IC8.6
- net N$9: now also IC6.11, IC8.6; no longer IC8.13
Routing:
- net IN_5: track 184.5 -> 312.4 mm
- net N$4: track 0.00 -> 93.3 mm
- net N$8: track 32.8 -> 109.9 mm
- net IN_2: track 83.3 -> 159.9 mm, vias 1 -> 0
- net N$32: track 86.0 -> 14.8 mm
- net N$35: track 0.00 -> 61.9 mm
- net +5V: track 330.4 -> 389.9 mm, vias 1 -> 0
- net N$29: track 25.2 -> 76.5 mm
- net N$10: track 41.6 -> 92.5 mm, vias 1 -> 0
- net N$66: track 55.4 -> 105.5 mm
- net IN_0: track 70.7 -> 118.3 mm, vias 1 -> 0
- net N$82: track 0.00 -> 41.7 mm
- net N$3 (its old number): track 38.0 -> 0.00 mm, vias 1 -> 0
- net N$67: track 44.8 -> 81.7 mm
- net N$80: track 36.8 -> 0.00 mm
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
Commit message: FR/RS Board one of final update
Parts:
- added C2, C3, C4, C5, C6, C7, C8, C9: 100n, rcl:C025-025X050
- C1: value 1u -> 100n; device rcl:C050-035X075 -> rcl:C025-025X050
- R19, R24, R25, R28, R33, R34: value 15k -> 4.7k
- moved C1 93.0 mm to (17.5, 58.4)
- moved IC7 16.0 mm to (73.2, 31.2)
- moved IC8 13.2 mm to (35.8, 27.4)
- moved V1 11.4 mm to (58.4, 8.13)
- moved R15 8.68 mm to (89.7, -3.30)
- moved R25 8.45 mm to (79.2, -9.65)
- moved R8 8.12 mm to (45.5, 68.6)
- moved R2 8.03 mm to (81.3, 68.6)
- moved R10 7.96 mm to (28.2, 68.6)
- moved R12 7.89 mm to (10.7, 68.6)
- moved R4 7.89 mm to (99.6, 68.6)
- moved R6 7.82 mm to (64.3, 68.6)
- moved R35 7.79 mm to (98.0, -31.8)
- moved R1 7.62 mm to (76.2, 68.6)
- moved R11 7.62 mm to (5.08, 68.6)
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Connections:
- net +5V: now also C2.1, C3.1, C4.1, C5.1, C6.1, C7.1, C8.1, C9.1
- net GND: now also C2.2, C3.2, C4.2, C5.2, C6.2, C7.2, C8.2, C9.2
Routing:
- net N$8: track 109.9 -> 87.1 mm
- net N$29: track 76.5 -> 57.7 mm
- net N$4: track 93.3 -> 110.4 mm
- net IN_1: track 81.2 -> 66.5 mm
- net N$1: track 44.6 -> 58.9 mm
- net N$2: track 24.1 -> 38.4 mm
- net IN_0: track 118.3 -> 105.6 mm
- net N$34: track 88.2 -> 77.3 mm
- net IN_5: track 312.4 -> 302.4 mm
- net FREQ3: track 21.5 -> 30.7 mm
- net N$3: track 17.2 -> 26.0 mm
- net N$66: track 105.5 -> 97.0 mm
- net IN_2: track 159.9 -> 151.4 mm
- net N$13: track 25.1 -> 16.6 mm
- net N$7: track 22.5 -> 29.5 mm
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Other:
- board size 114.3 x 169.8 mm -> 108.4 x 161.7 mm

Commit message: final version of FR/RS board
i think :)
Parts:
- moved C5 1.14 mm to (104.6, 66.0)
Routing:
- net +5V: track 395.7 -> 404.3 mm
Other:
- board size 108.4 x 161.7 mm -> 108.4 x 161.5 mm
Changed lines of the file:
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@@
 <plain>
 <wire x1="0" y1="-68.58" x2="108.438" y2="-68.58" width="0" layer="20"/>
-<wire x1="108.438" y1="-68.58" x2="108.438" y2="93.142" width="0" layer="20"/>
-<wire x1="108.438" y1="93.142" x2="0" y2="92.38" width="0" layer="20"/>
-<wire x1="0" y1="92.38" x2="0" y2="-68.58" width="0" layer="20"/>
-<dimension x1="3.79" y1="-40.64" x2="11.43" y2="-40.64" x3="7.61" y3="-40.64" textsize="1.778" layer="1"/>
+<wire x1="108.438" y1="-68.58" x2="108.438" y2="92.888" width="0" layer="20"/>
+<wire x1="108.438" y1="92.888" x2="0" y2="92.888" width="0" layer="20"/>
+<wire x1="0" y1="92.888" x2="0" y2="-68.58" width="0" layer="20"/>
 </plain>
 <attributes>
@@
 <attribute name="VALUE" x="73.914" y="56.134" size="1.27" layer="27" ratio="10" rot="R90"/>
 </element>
-<element name="C5" library="rcl" library_urn="urn:adsk.eagle:library:334" package="C025-025X050" package3d_urn="urn:adsk.eagle:package:23629/2" value="100n" x="105.664" y="65.532" smashed="yes" rot="R90">
-<attribute name="NAME" x="104.14" y="63.246" size="1.27" layer="25" ratio="10" rot="R90"/>
-<attribute name="SPICEPREFIX" value="C" x="105.664" y="65.532" size="1.778" layer="27" rot="R90" display="off"/>
-<attribute name="VALUE" x="108.458" y="63.246" size="1.27" layer="27" ratio="10" rot="R90"/>
+<element name="C5" library="rcl" library_urn="urn:adsk.eagle:library:334" package="C025-025X050" package3d_urn="urn:adsk.eagle:package:23629/2" value="100n" x="104.648" y="66.04" smashed="yes" rot="R90">
+<attribute name="NAME" x="103.124" y="63.754" size="1.27" layer="25" ratio="10" rot="R90"/>
+<attribute name="SPICEPREFIX" value="C" x="104.648" y="66.04" size="1.778" layer="27" rot="R90" display="off"/>
+<attribute name="VALUE" x="107.442" y="63.754" size="1.27" layer="27" ratio="10" rot="R90"/>
 </element>
 <element name="C6" library="rcl" library_urn="urn:adsk.eagle:library:334" package="C025-025X050" package3d_urn="urn:adsk.eagle:package:23629/2" value="100n" x="88.138" y="58.42" smashed="yes" rot="R90">
@@
 <wire x1="22.4155" y1="63.8175" x2="19.558" y2="60.96" width="0.2032" layer="1"/>
 <wire x1="104.668" y1="6.43" x2="106.934" y2="8.696" width="0.2032" layer="1"/>
-<wire x1="101.6" y1="57.15" x2="101.6" y2="57.277" width="0.2032" layer="1"/>
-<wire x1="106.3625" y1="59.436" x2="102.0445" y2="63.754" width="0.2032" layer="1"/>
 <wire x1="39.0525" y1="62.5475" x2="40.513" y2="64.008" width="0.2032" layer="1"/>
 <wire x1="40.513" y1="64.008" x2="47.244" y2="64.008" width="0.2032" layer="1"/>
@@
 <wire x1="82.1436" y1="28.8036" x2="94.1483375" y2="28.8036" width="0.2032" layer="1"/>
 <wire x1="94.1483375" y1="28.8036" x2="106.3625" y2="41.0177625" width="0.2032" layer="1"/>
-<wire x1="106.3625" y1="41.0177625" x2="106.3625" y2="59.436" width="0.2032" layer="1"/>
 <wire x1="54.61" y1="60.96" x2="57.4675" y2="63.8175" width="0.2032" layer="1"/>
 <wire x1="57.4675" y1="63.8175" x2="65.2145" y2="63.8175" width="0.2032" layer="1"/>
@@
 <wire x1="73.66" y1="59.69" x2="73.66" y2="61.722" width="0.2032" layer="1"/>
 <wire x1="73.66" y1="61.722" x2="75.7555" y2="63.8175" width="0.2032" layer="1"/>
-<wire x1="95.123" y1="63.754" x2="102.0445" y2="63.754" width="0.2032" layer="1"/>
 <wire x1="95.123" y1="63.754" x2="92.202" y2="63.754" width="0.2032" layer="1"/>
 <wire x1="90.424" y1="61.976" x2="92.202" y2="63.754" width="0.2032" layer="1"/>
-<wire x1="101.6" y1="57.277" x2="95.123" y2="63.754" width="0.2032" layer="1"/>
 <wire x1="34.8615" y1="58.166" x2="36.576" y2="58.166" width="0.2032" layer="1"/>
 <wire x1="29.21" y1="63.8175" x2="34.8615" y2="58.166" width="0.2032" layer="1"/>
-<wire x1="105.156" y1="63.754" x2="102.0445" y2="63.754" width="0.2032" layer="1"/>
 <contactref element="C1" pad="1"/>
 <wire x1="12.7" y1="57.15" x2="17.526" y2="57.15" width="0.2032" layer="1"/>
@@
 <wire x1="69.342" y1="58.42" x2="72.39" y2="58.42" width="0.2032" layer="1"/>
 <contactref element="C5" pad="1"/>
-<wire x1="105.664" y1="64.262" x2="105.156" y2="63.754" width="0.2032" layer="1"/>
 <contactref element="C6" pad="1"/>
 <wire x1="88.138" y1="57.15" x2="89.154" y2="58.166" width="0.2032" layer="1"/>
@@
 <wire x1="62.23" y1="22.098" x2="62.366025" y2="22.234025" width="0.2032" layer="1"/>
 <wire x1="62.366025" y1="22.234025" x2="66.665971875" y2="22.234025" width="0.2032" layer="1"/>
+<wire x1="97.155" y1="65.786" x2="95.123" y2="63.754" width="0.2032" layer="1"/>
+<wire x1="106.3625" y1="41.0177625" x2="106.3625" y2="63.5" width="0.2032" layer="1"/>
+<wire x1="106.3625" y1="63.5" x2="106.3625" y2="64.8335" width="0.2032" layer="1"/>
+<wire x1="106.3625" y1="64.8335" x2="105.41" y2="65.786" width="0.2032" layer="1"/>
+<wire x1="105.41" y1="65.786" x2="97.155" y2="65.786" width="0.2032" layer="1"/>
+<wire x1="101.6" y1="57.15" x2="98.044" y2="60.706" width="0.2032" layer="1"/>
+<wire x1="98.044" y1="60.706" x2="98.044" y2="62.992" width="0.2032" layer="1"/>
+<wire x1="98.044" y1="62.992" x2="99.822" y2="64.77" width="0.2032" layer="1"/>
+<wire x1="99.822" y1="64.77" x2="104.648" y2="64.77" width="0.2032" layer="1"/>
+<wire x1="104.648" y1="64.77" x2="105.0925" y2="64.77" width="0.2032" layer="1"/>
+<wire x1="105.0925" y1="64.77" x2="106.3625" y2="63.5" width="0.2032" layer="1"/>
 </signal>
 <signal name="GND">
@@
 <vertex x="-1.27" y="95.25"/>
 <vertex x="-1.524" y="-72.39"/>
-<vertex x="-1.524" y="-72.39"/>
-<vertex x="115.57" y="-72.39"/>
-<vertex x="115.57" y="95.25"/>
+<vertex x="110.49" y="-72.39"/>
+<vertex x="110.49" y="95.25"/>
 </polygon>
 <contactref element="C1" pad="2"/>
@@
 <contactref element="R17" pad="2"/>
 <contactref element="R33" pad="1"/>
-<contactref element="X13" pad="1"/>
 <wire x1="3.79" y1="-35.64" x2="17.7" y2="-35.64" width="0.2032" layer="1"/>
 <wire x1="17.7" y1="-35.64" x2="24.13" y2="-29.21" width="0.2032" layer="1"/>
 <wire x1="24.13" y1="-29.21" x2="26.67" y2="-29.21" width="0.2032" layer="1"/>
+<contactref element="X13" pad="1"/>
 </signal>
 <signal name="N$76">
@@
 <contactref element="R18" pad="2"/>
 <contactref element="R34" pad="1"/>
-<contactref element="X13" pad="3"/>
 <wire x1="26.67" y1="-40.64" x2="24.13" y2="-40.64" width="0.2032" layer="1"/>
 <wire x1="24.13" y1="-40.64" x2="19.13" y2="-45.64" width="0.2032" layer="1"/>
 <wire x1="19.13" y1="-45.64" x2="3.79" y2="-45.64" width="0.2032" layer="1"/>
+<contactref element="X13" pad="3"/>
 </signal>
 <signal name="N$78">
