Commit message: update rover model

File: rover_gazebo/models/rover/rover.urdf (robot description, URDF)
Before this commit: robot rover, 12 links, 11 joints
Joints:
- joint camera_joint: origin xyz=-0.28996  0       0.61032 rpy=0  0  3.14159265 -> xyz=-0.28996  0       0.61032 rpy=0  0.0873  3.14159265
- joint lidar_joint: origin xyz=0       0       0.64032 rpy=0  0  0 -> xyz=-0.28996       0       0.63032 rpy=0  0.1222  3.14159265

Commit message: delete collisions

File: rover_gazebo/models/rover/rover.urdf (robot description, URDF)
Before this commit: robot rover, 12 links, 11 joints
Joints:
- joint right_wheel_3_hinge: axis 0 -1  0 -> 0 1  0

Commit message: something

File: rover_gazebo/models/rover/rover.urdf (robot description, URDF)
Before this commit: robot rover, 12 links, 11 joints
Links:
- link camera_link: mass 0.1 -> 1
- link chassis: mass 5.0 -> 1.0
- link imu_link: mass 0.1 -> 1
- link left_steer: mass .2 -> 1
- link left_wheel_1: mass .2 -> 1
- link left_wheel_2: mass .2 -> 1
- link left_wheel_3: mass .2 -> 1
- link lidar_link: mass 0.1 -> 1
- link right_steer: mass .2 -> 1
- link right_wheel_1: mass .2 -> 1
- link right_wheel_2: mass .2 -> 1
- link right_wheel_3: mass .2 -> 1
Joints:
- joint left_steer_hinge: type continuous -> revolute
- joint left_wheel_1_hinge: limit lower=-9999999999999 upper=9999999999999 effort=0 velocity=0 -> effort=0 velocity=0
- joint left_wheel_2_hinge: limit lower=-9999999999999 upper=9999999999999 effort=0 velocity=0 -> effort=0 velocity=0
- joint left_wheel_3_hinge: limit lower=-9999999999999 upper=9999999999999 effort=0 velocity=0 -> effort=0 velocity=0
- joint right_steer_hinge: limit lower=-0.5 upper=1.0 effort=0.0 velocity=0.0 -> lower=-1. upper=0.5 effort=0.0 velocity=0.0; type continuous -> revolute
- joint right_wheel_1_hinge: limit lower=-9999999999999 upper=9999999999999 effort=0 velocity=0 -> effort=0 velocity=0
- joint right_wheel_2_hinge: limit lower=-9999999999999 upper=9999999999999 effort=0 velocity=0 -> effort=0 velocity=0
- joint right_wheel_3_hinge: limit lower=-9999999999999 upper=9999999999999 effort=0 velocity=0 -> effort=0 velocity=0

Commit message: better movement

File: rover_gazebo/models/rover/rover.urdf (robot description, URDF)
Before this commit: robot rover, 12 links, 11 joints
Links:
- link camera_link: mass 1 -> 0.1
- link chassis: mass 1.0 -> 5.0
- link imu_link: mass 1 -> 0.1
- link left_steer: mass 1 -> .2
- link left_wheel_1: mass 1 -> .2
- link left_wheel_2: mass 1 -> .2
- link left_wheel_3: mass 1 -> .2
- link lidar_link: mass 1 -> 0.1
- link right_steer: mass 1 -> .2
- link right_wheel_1: mass 1 -> .2
- link right_wheel_2: mass 1 -> .2
- link right_wheel_3: mass 1 -> .2
Joints:
- joint right_steer_hinge: limit lower=-1. upper=0.5 effort=0.0 velocity=0.0 -> lower=-1.0 upper=0.5 effort=0.0 velocity=0.0

Commit message: to check update

File: rover_gazebo/models/rover/rover.urdf (robot description, URDF)
Before this commit: robot rover, 12 links, 11 joints
Links:
- link camera_link: mass 0.1 -> 1
- link chassis: mass 5.0 -> 10.0
- link imu_link: mass 0.1 -> 1
- link left_steer: mass .2 -> 1
- link left_wheel_1: mass .2 -> 1
- link left_wheel_2: mass .2 -> 1
- link left_wheel_3: mass .2 -> 1
- link lidar_link: mass 0.1 -> 1
- link right_steer: mass .2 -> 1
- link right_wheel_1: mass .2 -> 1
- link right_wheel_2: mass .2 -> 1
- link right_wheel_3: mass .2 -> 1

Commit message: new version

File: rover_gazebo/models/rover/rover.urdf (robot description, URDF)
Before this commit: robot rover, 12 links, 11 joints
Links:
- link chassis: mass 10.0 -> 1.0
Joints:
- joint left_wheel_3_hinge: axis 0 1  0 -> 0 -1  0
- joint right_steer_hinge: limit lower=-1.0 upper=0.5 effort=0.0 velocity=0.0 -> lower=-1. upper=0.5 effort=0.0 velocity=0.0
