Commit message: working sphere

File: rover_gazebo/models/sphere/sphere.urdf (robot description, URDF)
Before this commit: robot sphere, 2 links, 1 joints
Links:
- removed link base_footprint
- link base_link: geometry collision box size=0.2 0.2 0.2; visual box size=0.2 0.2 0.2
Joints:
- removed joint base_link_joint
